File: sdr/tx_amp.kicad_sch (KiCad schematic)
At the start: 11 parts, among them Q5 AO3400A, Q6 AO3401A, U9 AD8001AR

Commit message: Many fixes. Updated mixers to use the analog switches rather than discretes.
Parts:
- added C25: 0.5pF, symbol Device:C
- added C26: 100n, symbol Device:C
- added C27: 1n, symbol Device:C
- added R30, R31: 470, symbol Device:R
- added R32: 1, Resistor_SMD:R_0402_1005Metric, symbol Device:R
- R24, R26: value 50 -> 120
- R27: value 24 -> 220
Connections:
- net +5V: now also R32.2; no longer U9.7 (V+)
- net GND: now also C26.2, C27.2, R31.2; no longer U9.2 (-)
- net at R27.1, R28.1, U9.6: now also C25.1
- net at R24.1, R26.1: now also U9.2 (-); no longer R27.2, U9.3 (+)
- new net +5P: C26.1, C27.1, R30.1, R32.1, U9.7 (V+)
- new net V_BIAS: C25.2, R27.2, R30.2, R31.1, U9.3 (+)
Other:
- moved on the sheet: R24, R26
