File: sdr/tx_amp.kicad_sch (KiCad schematic)
At the start: 17 parts, among them Q5 AO3400A, Q6 AO3401A, U9 AD8001AR

Commit message: Complete layout
Parts:
- removed R26: 120, Resistor_SMD:R_0402_1005Metric, symbol Device:R
- C25, C26, C27: footprint (none) -> Capacitor_SMD:C_0402_1005Metric
- R30, R31: footprint (none) -> Resistor_SMD:R_0402_1005Metric
Connections:
- net I_IN renamed RF_IN
Changed lines of the file:
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@@
   (junction (at 99.06 86.36) (diameter 0) (color 0 0 0 0)
   )
-  (junction (at 95.25 100.33) (diameter 0) (color 0 0 0 0)
-  )
   (junction (at 186.69 96.52) (diameter 0) (color 0 0 0 0)
   )
@@
     (stroke (width 0) (type default))
   )
-  (wire (pts (xy 90.17 100.33) (xy 95.25 100.33))
+  (wire (pts (xy 90.17 100.33) (xy 101.6 100.33))
     (stroke (width 0) (type default))
   )
@@
     (stroke (width 0) (type default))
   )
-  (wire (pts (xy 95.25 100.33) (xy 95.25 110.49))
-    (stroke (width 0) (type default))
-  )
   (wire (pts (xy 186.69 96.52) (xy 186.69 113.03))
     (stroke (width 0) (type default))
   )
-  (wire (pts (xy 76.2 110.49) (xy 82.55 110.49))
-    (stroke (width 0) (type default))
-  )
   (wire (pts (xy 186.69 113.03) (xy 189.23 113.03))
     (stroke (width 0) (type default))
@@
     (stroke (width 0) (type default))
   )
-  (wire (pts (xy 95.25 100.33) (xy 101.6 100.33))
-    (stroke (width 0) (type default))
-  )
   (wire (pts (xy 196.85 96.52) (xy 222.25 96.52))
     (stroke (width 0) (type default))
@@
   )
   (wire (pts (xy 196.85 95.25) (xy 196.85 96.52))
-    (stroke (width 0) (type default))
-  )
-  (wire (pts (xy 95.25 110.49) (xy 90.17 110.49))
     (stroke (width 0) (type default))
   )
@@
     (effects (font (size 1.27 1.27)) (justify left))
   )
-  (hierarchical_label "Q_IN" (shape input) (at 76.2 110.49 180) (fields_autoplaced)
+  (hierarchical_label "RF_IN" (shape input) (at 76.2 100.33 180) (fields_autoplaced)
     (effects (font (size 1.27 1.27)) (justify right))
   )
-  (hierarchical_label "I_IN" (shape input) (at 76.2 100.33 180) (fields_autoplaced)
-    (effects (font (size 1.27 1.27)) (justify right))
-  )
   (symbol (lib_id "power:+5V") (at 196.85 74.93 0) (unit 1)
     (in_bom yes) (on_board yes) (dnp no) (fields_autoplaced)
@@
       (effects (font (size 1.27 1.27)) (justify left))
     )
-    (property "Footprint" "" (at 145.7452 118.11 0)
+    (property "Footprint" "Capacitor_SMD:C_0402_1005Metric" (at 145.7452 118.11 0)
       (effects (font (size 1.27 1.27)) hide)
     )
@@
       (effects (font (size 1.27 1.27)) (justify left))
     )
-    (property "Footprint" "" (at 103.632 45.72 90)
+    (property "Footprint" "Resistor_SMD:R_0402_1005Metric" (at 103.632 45.72 90)
       (effects (font (size 1.27 1.27)) hide)
     )
@@
       (effects (font (size 1.27 1.27)) (justify left))
     )
-    (property "Footprint" "" (at 103.632 53.34 90)
+    (property "Footprint" "Resistor_SMD:R_0402_1005Metric" (at 103.632 53.34 90)
       (effects (font (size 1.27 1.27)) hide)
     )
@@
         (path "/ee974380-b45b-4b16-8475-50e4e51dc6cf/5adb175a-98d0-409a-bc02-3db049d84ccc"
           (reference "#PWR060") (unit 1)
-        )
-      )
-    )
-  )
-  (symbol (lib_id "Device:R") (at 86.36 110.49 270) (unit 1)
-    (in_bom yes) (on_board yes) (dnp no) (fields_autoplaced)
-    (property "Reference" "R26" (at 86.36 104.14 90)
-      (effects (font (size 1.27 1.27)))
-    )
-    (property "Value" "120" (at 86.36 106.68 90)
-      (effects (font (size 1.27 1.27)))
-    )
-    (property "Footprint" "Resistor_SMD:R_0402_1005Metric" (at 86.36 108.712 90)
-      (effects (font (size 1.27 1.27)) hide)
-    )
-    (property "Datasheet" "~" (at 86.36 110.49 0)
-      (effects (font (size 1.27 1.27)) hide)
-    )
-    (pin "1")
-    (pin "2")
-    (instances
-      (project "sdr"
-        (path "/ee974380-b45b-4b16-8475-50e4e51dc6cf/5adb175a-98d0-409a-bc02-3db049d84ccc"
-          (reference "R26") (unit 1)
         )
       )
@@
       (effects (font (size 1.27 1.27)))
     )
-    (property "Footprint" "" (at 107.95 75.8952 0)
+    (property "Footprint" "Capacitor_SMD:C_0402_1005Metric" (at 107.95 75.8952 0)
       (effects (font (size 1.27 1.27)) hide)
     )
@@
       (effects (font (size 1.27 1.27)) (justify left))
     )
-    (property "Footprint" "" (at 136.8552 118.11 0)
-      (effects (font (size 1.27 1.27)) hide)
-    )
+    (property "Footprint" "Capacitor_SMD:C_0402_1005Metric" (at 136.8552 118.11 0)
+      (effects (font (size 1.27 1.27)) hide)
+    )

Commit message: First version 0.1 completed
Parts:
- removed U9: AD8001AR, Package_SO:SOIC-8_3.9x4.9mm_P1.27mm, symbol Amplifier_Operational:AD8001AR
- added U6: GS8091-TR, Package_TO_SOT_SMD:SOT-23-5, symbol Amplifier_Operational:ADA4610-1xRJ
- R23, R29: value 4.7 -> 10
Connections:
- net +5P: now also U6.5 (V+)
- net GND: now also U6.2 (V-)
- net V_BIAS: now also U6.3 (+)
- net at C25.1, R27.1, R28.1: now also U6.1
- net at R24.1: now also U6.4 (-)
Changed lines of the file:
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@@
+    )
+  )
+  (symbol (lib_id "Amplifier_Operational:ADA4610-1xRJ") (at 109.22 97.79 0) (unit 1)
+    (in_bom yes) (on_board yes) (dnp no) (fields_autoplaced)
+    (property "Reference" "U6" (at 121.92 94.3611 0)
+      (effects (font (size 1.27 1.27)))
+    )
+    (property "Value" "GS8091-TR" (at 121.92 96.9011 0)
+      (effects (font (size 1.27 1.27)))
+    )
+    (property "Footprint" "Package_TO_SOT_SMD:SOT-23-5" (at 106.68 102.87 0)
+      (effects (font (size 1.27 1.27)) (justify left) hide)
+    )
+    (property "Datasheet" "https://www.analog.com/media/en/technical-documentation/data-sheets/ADA4610-1_4610-2_4610-4.pdf" (at 109.22 92.71 0)
+      (effects (font (size 1.27 1.27)) hide)
+    )
+    (pin "2")
+    (pin "5")
+    (pin "1")
+    (pin "3")
+    (pin "4")
+    (instances
+      (project "sdr"
+        (path "/ee974380-b45b-4b16-8475-50e4e51dc6cf/5adb175a-98d0-409a-bc02-3db049d84ccc"
+          (reference "U6") (unit 1)
+        )
+      )
     )
   )
@@
   (symbol (lib_id "Device:R") (at 196.85 91.44 0) (unit 1)
     (in_bom yes) (on_board yes) (dnp no) (fields_autoplaced)
-    (property "Reference" "R29" (at 199.39 90.1699 0)
-      (effects (font (size 1.27 1.27)) (justify left))
-    )
-    (property "Value" "4.7" (at 199.39 92.7099 0)
+    (property "Reference" "R29" (at 199.39 90.805 0)
+      (effects (font (size 1.27 1.27)) (justify left))
+    )
+    (property "Value" "10" (at 199.39 93.345 0)
       (effects (font (size 1.27 1.27)) (justify left))
     )
@@
   (symbol (lib_id "Device:R") (at 196.85 101.6 0) (unit 1)
     (in_bom yes) (on_board yes) (dnp no) (fields_autoplaced)
-    (property "Reference" "R23" (at 199.39 100.3299 0)
-      (effects (font (size 1.27 1.27)) (justify left))
-    )
-    (property "Value" "4.7" (at 199.39 102.8699 0)
+    (property "Reference" "R23" (at 199.39 100.965 0)
+      (effects (font (size 1.27 1.27)) (justify left))
+    )
+    (property "Value" "10" (at 199.39 103.505 0)
       (effects (font (size 1.27 1.27)) (justify left))
     )
@@
         )
       )
-    )
-  )
-  (symbol (lib_id "Amplifier_Operational:AD8001AR") (at 109.22 97.79 0) (unit 1)
-    (in_bom yes) (on_board yes) (dnp no) (fields_autoplaced)
-    (property "Reference" "U9" (at 120.65 93.091 0)
-      (effects (font (size 1.27 1.27)))
-    )
-    (property "Value" "AD8001AR" (at 120.65 95.631 0)
-      (effects (font (size 1.27 1.27)))
-    )
-    (property "Footprint" "Package_SO:SOIC-8_3.9x4.9mm_P1.27mm" (at 106.68 102.87 0)
-      (effects (font (size 1.27 1.27)) (justify left) hide)
-    )
-    (property "Datasheet" "https://www.analog.com/media/en/technical-documentation/data-sheets/ad8001.pdf" (at 113.03 93.98 0)
-      (effects (font (size 1.27 1.27)) hide)
-    )
-    (pin "1")
-    (pin "2")
-    (pin "3")
-    (pin "4")
-    (pin "5")
-    (pin "6")
-    (pin "7")
-    (pin "8")
-    (instances
-      (project "sdr"
-        (path "/ee974380-b45b-4b16-8475-50e4e51dc6cf/5adb175a-98d0-409a-bc02-3db049d84ccc"
-          (reference "U9") (unit 1)
-        )
-      )
