File: sdr/sdr.kicad_sch (KiCad schematic)
At the start: 7 parts, among them J3 Conn_Coaxial, U10 BGA2817, U5 BGA2817, U6 NC7SB3157L6X, U8 FM1630C

Commit message: Complete layout
Parts:
- removed U6: NC7SB3157L6X, Package_SON:Fairchild_MicroPak-6_1.0x1.45mm_P0.5mm, symbol Analog_Switch:NC7SB3157L6X
- added R6: 0, Resistor_SMD:R_0402_1005Metric, symbol Device:R
- added TP2: TMIX, TestPoint:TestPoint_Keystone_5015_Micro-Minature, symbol Connector:TestPoint_Flag
- TP4: value RF_IN -> RX; footprint TestPoint:TestPoint_Pad_D1.0mm -> TestPoint:TestPoint_Keystone_5015_Micro-Minature
- TP5: value RF_OUT -> TX; footprint TestPoint:TestPoint_Pad_D1.0mm -> TestPoint:TestPoint_Keystone_5015_Micro-Minature
Connections:
- new net TX Amplifier/RF_IN: R6.2
- new net Tx Mixers/RF_OUT: R6.1, TP2.1
Other:
- sheet TX Amplifier ports: added RF_IN; removed I_IN, Q_IN
- sheet Tx Mixers ports: added RF_OUT; removed RF_I, RF_Q
