File: sdr/usb_power.kicad_sch (KiCad schematic)
At the start: 9 parts, among them J1 USB_C_Receptacle_USB2.0, U1 AMS1117-3.3

Commit message: Update the via size. Reduce footprints outside board.
Parts:
- FB1: value BLM18KG221SN1D -> GZ2012D101TF; footprint Inductor_SMD:L_0603_1608Metric -> Inductor_SMD:L_0805_2012Metric; LCSC C88980 -> (none)
Changed lines of the file:
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@@
     )
   )
-  (symbol (lib_name "+5V_1") (lib_id "power:+5V") (at 208.28 73.66 0) (unit 1)
+  (symbol (lib_id "power:+5V") (at 208.28 73.66 0) (unit 1)
     (in_bom yes) (on_board yes) (dnp no) (fields_autoplaced)
     (property "Reference" "#PWR06" (at 208.28 77.47 0)
@@
       (effects (font (size 1.27 1.27)))
     )
-    (property "Value" "BLM18KG221SN1D" (at 164.4142 66.675 90)
-      (effects (font (size 1.27 1.27)))
-    )
-    (property "Footprint" "Inductor_SMD:L_0603_1608Metric" (at 164.465 73.533 90)
+    (property "Value" "GZ2012D101TF" (at 164.4142 66.675 90)
+      (effects (font (size 1.27 1.27)))
+    )
+    (property "Footprint" "Inductor_SMD:L_0805_2012Metric" (at 164.465 73.533 90)
       (effects (font (size 1.27 1.27)) hide)
     )
@@
       (effects (font (size 1.27 1.27)) hide)
     )
-    (property "LCSC" "C88980" (at 164.465 71.755 90)
-      (effects (font (size 1.27 1.27)) hide)
-    )
+    (property "LCSC" "" (at 164.465 71.755 90)
+      (effects (font (size 1.27 1.27)) hide)
+    )
